File: OpenEVSE_PLUS_v4/OpenEVSE_PLUS_v4.brd (EAGLE design)
At the start: 65.3 x 44.9 mm, 77 parts, among them IC1 MID400, IC2 MEGA8-AI, IC3 LMV358, IC4 LMV358, IC5 AQH1213, IC6 MID400, Q1 16000, Q2 2222A, Q3 2222A

Commit message: Updates to components
Updated parts values so generic footprints report the correct part when exporting Eagle generated BOM.

IC2 value 328P 
IC3 value LM358 
IC4 value LF353
TVS value P6SMB16CA
D1 value AZ23C5V6-7-F

DC/DC value MD112D-12E
Parts:
- D1: value BAS40-06 -> AZ23C5V6-7-F
- DCDC: value D107E -> MD112D-12E
- IC2: value MEGA8-AI -> ATMEGA328P-AU
- IC3: value LMV358 -> LM358
- IC4: value LMV358 -> LF353
- R1: value 650 -> 620
- R26: value 28 -> 22
- TVS: value P6SMB16A -> P6SMB16CA
Changed lines of the file:
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@@
 <?xml version="1.0" encoding="utf-8"?>
 <!DOCTYPE eagle SYSTEM "eagle.dtd">
-<eagle version="7.1.0">
+<eagle version="7.3.0">
 <drawing>
 <settings>
@@
 <elements>
 <element name="ISP1" library="adafruit" package="AVRISP" value="AVRISP-6" x="40.3062" y="40.649" rot="MR180"/>
-<element name="IC2" library="atmel" package="TQFP32-08" value="MEGA8-AI" x="19.529" y="21.472" rot="R90">
+<element name="IC2" library="atmel" package="TQFP32-08" value="ATMEGA328P-AU" x="19.529" y="21.472" rot="R90">
 <attribute name="MF" value="" x="19.529" y="21.472" size="1.778" layer="27" rot="R90" display="off"/>
 <attribute name="MPN" value="ATMEGA8-16AU" x="19.529" y="21.472" size="1.778" layer="27" rot="R90" display="off"/>
@@
 <attribute name="OC_NEWARK" value="73M8863" x="19.529" y="21.472" size="1.778" layer="27" rot="R90" display="off"/>
 </element>
-<element name="IC4" library="SparkFun" package="SO08" value="LMV358" x="26.641" y="33.918" rot="R270"/>
+<element name="IC4" library="SparkFun" package="SO08" value="LF353" x="26.641" y="33.918" rot="R270"/>
 <element name="C12" library="SparkFun" package="0805" value=".1uf" x="18.985" y="28.5004" rot="R90"/>
 <element name="C1" library="SparkFun" package="0805" value="22pf" x="30.2514" y="18.5114" rot="R270"/>
@@
 <element name="R12" library="SparkFun" package="0805" value="2.4k" x="26.924" y="42.235" rot="R90"/>
 <element name="R13" library="SparkFun" package="0805" value="2.4k" x="32.258" y="42.22" rot="R270"/>
-<element name="R1" library="SparkFun" package="0805" value="650" x="20.137" y="35.687"/>
+<element name="R1" library="SparkFun" package="0805" value="620" x="20.137" y="35.687"/>
 <element name="R5" library="SparkFun" package="0805" value="56k" x="15.946" y="30.861"/>
 <element name="R6" library="SparkFun" package="0805" value="100k" x="15.946" y="33.274"/>
@@
 <element name="R10" library="SparkFun" package="0805" value="10k" x="15.875" y="28.519"/>
 <element name="R11" library="SparkFun" package="0805" value="330" x="10.1092" y="24.9884" rot="R90"/>
-<element name="IC3" library="SparkFun" package="SO08" value="LMV358" x="25.7556" y="10.16" rot="R90"/>
+<element name="IC3" library="SparkFun" package="SO08" value="LM358" x="25.7556" y="10.16" rot="R90"/>
 <element name="C14" library="SparkFun" package="EIA3216" value="10uf" x="19.558" y="5.7912"/>
-<element name="D1" library="diode" package="SOT23" value="BAS40-06" x="12.4206" y="11.0744" rot="R270"/>
+<element name="D1" library="diode" package="SOT23" value="AZ23C5V6-7-F" x="12.4206" y="11.0744" rot="R270"/>
 <element name="C7" library="SparkFun" package="0805" value=".1uf" x="25.7556" y="2.9972" rot="R90"/>
 <element name="R14" library="SparkFun" package="0805" value="100k" x="19.7104" y="10.8712"/>
@@
 <element name="R20" library="SparkFun" package="0805" value="1k" x="22.9616" y="2.7686" rot="R180"/>
 <element name="Q1" library="adafruit" package="NX3225" value="16000" x="27.5336" y="18.3642" rot="R270"/>
-<element name="DCDC" library="Qxd" package="DCDC_SIP" value="D107E" x="19.5834" y="39.2176" rot="MR180"/>
+<element name="DCDC" library="Qxd" package="DCDC_SIP" value="MD112D-12E" x="19.5834" y="39.2176" rot="MR180"/>
 <element name="D2" library="diode" package="SOD123" value="1N4148" x="6.7564" y="19.9644" rot="R90"/>
 <element name="D3" library="diode" package="SOD123" value="1N4148" x="27.6606" y="5.9182"/>
 <element name="D4" library="diode" package="SOD123" value="1N4148" x="18.2118" y="3.0226"/>
-<element name="TVS" library="diode" package="SMB" value="P6SMB16A" x="7.5692" y="30.8356" rot="R270"/>
+<element name="TVS" library="diode" package="SMB" value="P6SMB16CA" x="7.5692" y="30.8356" rot="R270"/>
 <element name="Q3" library="transistor-npn" package="SOT23" value="2222A" x="6.9088" y="25.0698" rot="R90"/>
 <element name="LOGO1" library="ohw-logo" package="OSHW_8X150_NOTEXT" value="OSHW_LOGO_8MILX0150-NT" x="48.0568" y="3.937"/>
@@
 <element name="R21" library="SparkFun" package="0805" value="100k" x="13.208" y="5.1816" rot="R270"/>
 <element name="R25" library="SparkFun" package="0805" value="100k" x="16.6116" y="10.8712" rot="R180"/>
-<element name="R26" library="SparkFun" package="0805" value="28" x="11.2268" y="5.1816" rot="R270"/>
+<element name="R26" library="SparkFun" package="0805" value="22" x="11.2268" y="5.1816" rot="R270"/>
 <element name="A_CT" library="SparkFun" package="1X02" value="" x="8.5598" y="5.6642" rot="MR270"/>
 <element name="C8" library="SparkFun" package="0805" value=".1uf" x="23.876" y="15.9512" rot="R90"/>
