File: OpenEVSE_PLUS_v5/OpenEVSE_PLUS_v5.sch (EAGLE design)
At the start: 71 parts, among them IC1 HCPL-2731, IC2 MEGA8-AI, IC3 LMV358, IC4 LMV358, IC5 AQH1213, Q1 16000, Q2 2222A, Q3 2222A

Commit message: v5
V5 files added
Parts:
- removed AC_LINE, AC_RELAY, AC_TEST: TE 1776275-2, SparkFun:M023.5MM_LOCK
- removed A_CT: (no value), SparkFun:M02PTH
- removed G_CT: G_CT, SparkFun:M04LOCK
- removed RELAY: (no value), SparkFun:M03SCREW_LOCK
- added 12VDC: (no value), SparkFun-Connectors:M023.5MM
- added AC: JST-VH-6, OpenEVSE:JST-VH-6
- added AMP_CT: AMP_CT, OpenEVSE:MOLEX_2
- added DC_RELAY: DC_RELAY, OpenEVSE:MOLEX_3
- added GFCI_CT: GFCI_CT, OpenEVSE:GFCI_4
- added R12, R13: 2.4k, SparkFun:RESISTOR0805-RES
- added R28: 180, rcl:R-US_R1206
- added U$1: MOV, OpenEVSE:MOV
- added U$3, U$4: HOLE, OpenEVSE:HOLE
- D1: value BAS40-06 -> AZ23C5V6-7-F
- DCDC: value D107E -> MD112D-12E
- IC2: value MEGA8-AI -> ATMEGA328P-AU
- IC3: value LMV358 -> LM358
- IC4: value LMV358 -> LF353
- PILOT: value Pilot -> (none); device SparkFun:M03SCREW_LOCK -> SparkFun-Connectors:M023.5MM
- PS1: value AAF-05 -> MPM-04E-1205; device Qxd:AAF-05 -> Qxd:MPM-04E-1205
- R1: value 650 -> 620
- R17: value GND -> 412
- R22: value 200k -> 200K
- R26: value 28 -> 22
- TVS: value P6SMB16A -> P6SMB16CA
Connections:
- removed net N$12 (its old number): AC_LINE.1, F2.P$1
- removed net N$13 (its old number): AC_LINE.2, F1.P$1
- removed net N$17 (its old number): AC_TEST.1, R4.1
- removed net N$29: AC_TEST.2, R22.1
- new net +12V: 12VDC.2, C13.1, D2.C, D5.C, DCDC.VIN+, DC_RELAY.2, PS1.12V
- new net ACIN1: AC.1, F2.P$1
- new net ACIN2: AC.2, AC.3, F1.P$1, U$1.1
- new net ACTEST1: AC.6, R4.1
- new net ACTEST2: AC.5, R22.1
- net +5V: now also PS1.5V, R28.2; no longer C13.1, D2.C, D5.C, DCDC.VIN+, PS1.P_OUT, RELAY.2
- net -12V: now also R12.1
- net 12V: now also R13.2
- net ACRELAY: now also AC.4, IC5.6, U$1.2; no longer AC_RELAY.1, IC5.8
- net AC_TEST: now also IC1.O1; no longer IC1.O2
- net AC_TEST_2: now also IC1.O2; no longer IC1.O1
- net AMP_READ: now also AMP_CT.2; no longer A_CT.1
- net FUSEL: now also IC5.8, PS1.ACH; no longer IC5.6, PS1.AC_L
- net FUSEN: now also PS1.ACN; no longer AC_RELAY.2, PS1.AC_N
- net GND: now also 12VDC.1, GFCI_CT.1, GFCI_CT.4, PS1.GND, R12.2, R13.1, R28.1, U$3.GND, U$4.GND; no longer G_CT.1, G_CT.4, PILOT.3, PS1.N_OUT
- net N$1: now also DC_RELAY.3; no longer RELAY.1
- net N$20: now also GFCI_CT.2; no longer G_CT.2
- net N$22: now also GFCI_CT.3; no longer G_CT.3
- net N$6: now also DC_RELAY.1; no longer RELAY.3
- net N$7: now also AMP_CT.1; no longer A_CT.2
- net PILOT: now also PILOT.1; no longer PILOT.2
- net PP: now also PILOT.2; no longer PILOT.1
Other:
- moved on the sheet: D7, D8, IC1
