File: OpenEVSE_PLUS_v5.5/OpenEVSE_PLUS_v5.5/OpenEVSE_PLUS_v5.5.kicad_pcb (KiCad board)
At the start: 2 copper layers, 65.4 x 45.8 mm, 78 parts, among them IC1 HCPL-2731, IC2 ATMEGA328P-AU, IC3 LM358, IC4 LF353, IC5 AQH1213, IC6 TC1044S, Q1 16000, Q2 2222A, Q3 2222A

Commit message: WIP new power module TMLM 04225
Parts:
- removed TVS0: P6SMB16CA, OpenEVSE_PLUS_v5.5:SMB
- PS1: value MPM-04E-1205 -> (none); footprint OpenEVSE_PLUS_v5.5:MPM-04E-1205 -> Converter_ACDC:Converter_ACDC_TRACO_TMLM-04_THT
- moved PS1 42.4 mm to (131.0, 92.5), turned to -90 degrees
- moved R25 2.28 mm to (134.0, 118.5)
- moved R7 1.99 mm to (131.8, 90.0)
- moved PILOT0 1.98 mm to (119.2, 96.0)
- moved D1 1.95 mm to (128.4, 116.0)
- moved R15 1.60 mm to (137.0, 119.5), turned to -90 degrees
- moved IC6 1.33 mm to (150.2, 88.6)
- moved R17 1.14 mm to (128.1, 119.0), turned to 180 degrees
- moved C5 0.79 mm to (152.1, 85.0)
- moved C14 0.77 mm to (136.3, 122.4)
- moved C7 0.77 mm to (142.4, 124.7)
- moved C9 0.77 mm to (140.1, 121.8)
- moved D3 0.77 mm to (144.3, 121.8)
- moved IC3 0.77 mm to (142.4, 117.5)
- moved R14 0.77 mm to (136.3, 116.8)
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Routing:
- net +5V: track 146.1 -> 204.8 mm
- net +12V: track 80.7 -> 93.1 mm, vias 0 -> 1
- net PILOT: track 28.4 -> 20.9 mm
- net GFCI_INT: track 19.0 -> 24.1 mm
- net AMP_READ: track 32.9 -> 36.9 mm
- net FUSEL: track 26.7 -> 23.5 mm
- net N$23: track 26.0 -> 23.8 mm
- net PILOTREAD: track 16.3 -> 18.0 mm
- net -12V: track 16.1 -> 14.7 mm
- net PP: track 44.2 -> 45.6 mm
- net N$19: track 6.73 -> 5.63 mm
- net PWM: track 14.8 -> 13.8 mm
- net N$7: track 16.9 -> 15.9 mm
- net N$6: track 14.8 -> 13.9 mm
- net ACTEST2: track 10.4 -> 9.62 mm
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Other:
- board text added: "v5.5.PWR"
- board text removed: "v5.5"
